File: Dronic.kicad_sch (KiCad schematic)
At the start: 55 parts, among them J1 Screw_Terminal_01x02, J2 Screw_Terminal_01x02, SW1 SW_Push, SW2 SW_Push, U1 RP2040, U2 2137160001, U3 W25Q128JVS, U4 LTC3521EFE-PBF, U5 AP62150WU, U6 ECH8690-TL-H, U8 NTJD5121NT1G, Y1 ABM3B-12.000MHZ-10-1-U-T

Commit message: SM06B-SRSS-TB 6 Pin Connector Male, this will be used for the Benewake TFS20-L LiDAR Module
Parts:
- J1: value Screw_Terminal_01x02 -> SWDIO_PH_TERM
Other:
- note added: "Add a fuse after limiting calculations."
- note added: "VOUT 5V - 1.6A MAX"
- note removed: ""
- note removed: "VOUT 5V - 1.6A"
- moved on the sheet: C1, C13, C14, C2, C3, D1, D2, D3, D4, J2, L1, L2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

Commit message: Schematic Updates
Parts:
- added J3: JST_SH_6P_1.00mm, Connector_JST:JST_SH_SM06B-SRSS-TB_1x06-1MP_P1.00mm_Horizontal, symbol Connector:Conn_01x06_Pin
- L4: value 71uH -> 68uH; footprint Inductor_SMD:L_0402_1005Metric -> Inductor_SMD:L_Bourns-SRR1005
- R20, R21: value 10K -> 5K
Connections:
- net +3.3V: now also J3.1 (Pin_1), J3.2 (Pin_2)
- net GND: now also J3.6 (Pin_6)
- net SCL: now also J3.4 (Pin_4)
- net SDA: now also J3.3 (Pin_3)
- net TFS20_CS: now reaches U1.13 (GPIO10)
- net TFS20_CS: now also J3.5 (Pin_5)
Other:
- moved on the sheet: C1, C10, C11, C12, C13, C14, C2, C3, C4, C5, C6, C7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
