File: Dronic.kicad_sch (KiCad schematic)
At the start: 112 parts, among them IC1 ACS71240LLCBTR-050U5, IC10 ACS71240LLCBTR-050U5, IC11 ACS71240LLCBTR-050U5, IC12 ACS71240LLCBTR-050U5, IC13 XBP9B-XCWT-001, IC2 ACS71240LLCBTR-050U5, IC3 ACS71240LLCBTR-050U5, IC4 ACS71240LLCBTR-050U5, IC5 ACS71240LLCBTR-050U5, IC6 ACS71240LLCBTR-050U5, IC7 ACS71240LLCBTR-050U5, IC8 ACS71240LLCBTR-050U5, IC9 ACS71240LLCBTR-050U5, J1 SWDIO_PH_TERM, J2 Screw_Terminal_01x02, J3 JST_SH_6P_1.00mm, J4 Screw_Terminal_01x03, J5 Screw_Terminal_01x03, J6 Screw_Terminal_01x03, J7 Screw_Terminal_01x03, Q1 Q_NMOS, Q10 Q_NMOS, Q11 Q_NMOS, Q12 Q_NMOS, Q13 Q_NMOS, Q14 Q_NMOS, Q15 Q_NMOS, Q16 Q_NMOS, Q17 Q_NMOS, Q18 Q_NMOS, Q19 Q_NMOS, Q2 Q_NMOS, Q20 Q_NMOS, Q21 Q_NMOS, Q22 Q_NMOS, Q23 Q_NMOS, Q24 Q_NMOS, Q25 Q_NMOS, Q26 Q_NMOS, Q27 Q_NMOS, Q28 Q_NMOS, Q3 Q_NMOS, Q4 Q_NMOS, Q5 Q_NMOS, Q6 Q_NMOS, Q7 Q_NMOS, Q8 Q_NMOS, Q9 Q_NMOS, SW1 SW_Push, SW2 SW_Push, U1 RP2040, U10 MAX11616, U2 2137160001, U3 W25Q128JVS, U4 LTC3521EFE-PBF, U5 AP62150WU, U6 ECH8690-TL-H, U7 PCF8575DBR, U8 NTJD5121NT1G, U9 PCF8575DBR, Y1 ABM3B-12.000MHZ-10-1-U-T

Commit message: Edits
Connections:
- net SCL: now also U1.7 (GPIO5); no longer U1.12 (GPIO9)
- net SDA: now also U1.6 (GPIO4); no longer U1.11 (GPIO8)
Other:
- moved on the sheet: R20, R21
Changed lines of the file:
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@@
 	)
 	(rectangle
+		(start 447.04 121.92)
+		(end 571.5 187.96)
+		(stroke
+			(width 0.762)
+			(type solid)
+		)
+		(fill
+			(type none)
+		)
+	)
+	(rectangle
 		(start 35.56 40.64)
 		(end 60.96 68.58)
@@
 	)
 	(junction
-		(at 336.55 72.39)
-		(diameter 0)
-		(color 0 0 0 0)
-	)
-	(junction
 		(at 92.71 306.07)
 		(diameter 0)
@@
 	)
 	(junction
-		(at 339.09 59.69)
+		(at 337.82 49.53)
 		(diameter 0)
 		(color 0 0 0 0)
@@
 	)
 	(junction
+		(at 335.28 62.23)
+		(diameter 0)
+		(color 0 0 0 0)
+	)
+	(junction
 		(at 124.46 247.65)
 		(diameter 0)
@@
 	)
 	(junction
-		(at 341.63 74.93)
-		(diameter 0)
-		(color 0 0 0 0)
-	)
-	(junction
 		(at 165.1 52.07)
 		(diameter 0)
@@
 		(color 0 0 0 0)
 	)
+	(junction
+		(at 340.36 64.77)
+		(diameter 0)
+		(color 0 0 0 0)
+	)
 	(no_connect
 		(at 95.25 260.35)
@@
 	(wire
 		(pts
-			(xy 339.09 59.69) (xy 336.55 59.69)
+			(xy 337.82 49.53) (xy 335.28 49.53)
 		)
 		(stroke
@@
 	(wire
 		(pts
+			(xy 320.04 62.23) (xy 335.28 62.23)
+		)
+		(stroke
+			(width 0)
+			(type default)
+		)
+	)
+	(wire
+		(pts
 			(xy 54.61 223.52) (xy 55.88 223.52)
 		)
@@
 	(wire
 		(pts
-			(xy 320.04 74.93) (xy 341.63 74.93)
-		)
-		(stroke
-			(width 0)
-			(type default)
-		)
-	)
-	(wire
-		(pts
 			(xy 120.65 52.07) (xy 123.19 52.07)
 		)
@@
 	(wire
 		(pts
-			(xy 336.55 72.39) (xy 349.25 72.39)
+			(xy 335.28 62.23) (xy 347.98 62.23)
 		)
 		(stroke
@@
 	(wire
 		(pts
+			(xy 320.04 64.77) (xy 340.36 64.77)
+		)
+		(stroke
+			(width 0)
+			(type default)
+		)
+	)
+	(wire
+		(pts
 			(xy 71.12 363.22) (xy 71.12 365.76)
 		)
@@
 	(wire
 		(pts
-			(xy 341.63 71.12) (xy 341.63 74.93)
+			(xy 340.36 60.96) (xy 340.36 64.77)
 		)
 		(stroke
@@
 	(wire
 		(pts
-			(xy 320.04 72.39) (xy 336.55 72.39)
-		)
-		(stroke
-			(width 0)
-			(type default)
-		)
-	)
-	(wire
-		(pts
 			(xy 48.26 251.46) (xy 49.53 251.46)
 		)
@@
 	(wire
 		(pts
-			(xy 339.09 59.69) (xy 341.63 59.69)
+			(xy 337.82 49.53) (xy 340.36 49.53)
 		)
 		(stroke
@@
 	(wire
 		(pts
-			(xy 341.63 74.93) (xy 349.25 74.93)
+			(xy 340.36 64.77) (xy 347.98 64.77)
 		)
 		(stroke
@@
 	(wire
 		(pts
-			(xy 341.63 59.69) (xy 341.63 63.5)
+			(xy 340.36 49.53) (xy 340.36 53.34)
 		)
 		(stroke
@@
 	(wire
 		(pts
-			(xy 336.55 71.12) (xy 336.55 72.39)
+			(xy 335.28 60.96) (xy 335.28 62.23)
 		)
 		(stroke
@@
 	(wire
 		(pts
-			(xy 336.55 59.69) (xy 336.55 63.5)
+			(xy 335.28 49.53) (xy 335.28 53.34)
 		)
 		(stroke
@@
 			"AAAAYBYgBwcAAAAAAAAAwA+xEgAAAAAAAAAAP8RKAAAAAAAAAAD8qEAgCPcYAAAAAAAAAADmCqwr"
 			"AQAAAAAAAADwQ6wEAAAAAAAAAMAPsRIAAAAAAAAAAD/ESgAAAAAAAAAA/BArAQAAAAAAAADwQ6wE"
-			"AAAAAAAAAMDv/wP93+DaMbEUewAAAABJRU5ErkJggg=="
+			"AAAAAAAAAMDv/wP93+DaMbEUewAAAABJRU5ErkJgggBQAFQAbgA0AFEAZwBoADMARABGADQAbgBX"
+			"AGkAdAA1ADgATABvAHAATwBsAE4ATgBXAGgANQBnAGQAcwAzAFIAUQBlADMAbQBzAGEATgBMAEwA"
+			"eQBjAG0AUAB2ADYAcwB2AGcAaABUAFQAVgBkADUAYwBVADMAcABEAHcAZgBOAHcAZgA5AC8AeQB2"
+			"AEUASQBzACsAUQBwAG8AbQByAGYAZABlADIAcgBOAGoAYQB2AEEAYgBaAHAAWgAxAGIAdgBzADYA"
+			"TgAvAEMASQArAHMATgAxAGIANQBjAFUAMwBaAEsAZwBqAEwAQwBmAGgAawBBADcAZgBHAEcAagBn"
+			"AFEAVAAzAG8AYwA3AHkAOAB2AEMAWgBNAG0AQgBBAFUARgBPAFQAaQA0AGoAWgBzADIAUABDAGcA"
+			"bwBDAEIASABSADAAYwBXADYAdwBVADcAbQBvAEgAKwB3AE0ATABDAHcAcwA3AE8ATABqAFEAMABk"
+			"AE8AegBZAGMAVAA0ACsAUABzAE8ARwBEAGYAZgAyADkAaABZAEsAaABTAFkAbQBKAGwAQwBiAEIA"
+			"ZwBBAEEAQQBBAEEAQQBkAEQAOQBaAFkAWABHADUAcABuAEYANABDADgALwBEAHoAZQBGAFoAMAB5"
+			"AHkAMgB5AFYAQwAwAGYARQBlAFcAZgBiAHgAcABEAEEANQBOAEcASgBYAFcAeABUAG8ASwBMAHkA"
+			"ZQBtAFcAYgBiAHEAMwBNAEgAaQBDADcAMQBRAGIAbwBHADAAZQBWAHAAeABoAGoAWABIAHYATgBW"
+			"AEMAMQBkAGQALwBTAGMANQB0AE4AMABiAG0ASwBVADUAdwBqAEoAUwBpAEsASQBvAG8AaQBBAHQA"
+			"dAA4ADUAYgBzAHkAeABBAHUARABjAE0AdwBtAHUAOABQAHgASQB4AGQANgBUAHQAbgBPADcAWQBM"
+			"AEgAbgBkAHcAOAArAEYAMQB1AEYANQBWAGEAVQBGAFIANQA1AHMAeQBnAEUAQwAvAEUAdABBAFgA"
+			"dQBiAG0ANQBSAFUAVgBGAGwAWgBRADgAOAB2AFEAVQBMAEYAagBRAGMAYQBFAGkAWQBCAHoAbwBk"
+			"AEwAcQBmAG4AeAArAFgAYQAvAG4ANABjAGUAVwA5AGUALwBmAGYAZQB1AHQAMQBLAHkAcwBZAGYA"
+			"UQBNAEEAQQBBAEEAQQBBAFAAbwAyAE0AbgAvAGYAawB2AGsASgBQAHQAdgAyAEsAZwBrAEIAQwA5"
+			"AGQAUAB4ADkAdQBkADYAMQBmAGsASgBPADAAbwBqAHoAagBnAC8AWABSAGkAUwBOAHcAdABZAEgA"
+			"NgBBAGIATQBQAFoAcgBNADgAQwBtACsAYwBQADcAbA=="
 		)
 	)
@@
 	(global_label "SCL"
 		(shape input)
-		(at 349.25 74.93 0)
+		(at 347.98 64.77 0)
 		(fields_autoplaced yes)
 		(effects
@@
 		)
 		(property "Intersheetrefs" "${INTERSHEET_REFS}"
-			(at 355.7428 74.93 0)
+			(at 354.4728 64.77 0)
 			(effects
 				(font
@@
 	(global_label "SDA"
 		(shape input)
-		(at 349.25 72.39 0)
+		(at 347.98 62.23 0)
 		(fields_autoplaced yes)
 		(effects
@@
 		)
 		(property "Intersheetrefs" "${INTERSHEET_REFS}"
-			(at 355.8033 72.39 0)
+			(at 354.5333 62.23 0)
 			(effects
 				(font
@@
 	(symbol
 		(lib_id "Device:R")
-		(at 341.63 67.31 0)
+		(at 340.36 57.15 0)
 		(unit 1)
 		(exclude_from_sim no)
@@
 		(dnp no)
 		(property "Reference" "R21"
-			(at 343.662 66.548 0)
+			(at 342.392 56.388 0)
 			(effects
 				(font
@@
 		)
 		(property "Value" "5K"
-			(at 343.408 68.834 0)
+			(at 342.138 58.674 0)
 			(effects
 				(font
@@
 		)
 		(property "Footprint" "Resistor_SMD:R_0402_1005Metric"
-			(at 339.852 67.31 90)
+			(at 338.582 57.15 90)
 			(effects
 				(font
@@
 		)
 		(property "Datasheet" "~"
-			(at 341.63 67.31 0)
+			(at 340.36 57.15 0)
 			(effects
 				(font
@@
 		)
 		(property "Description" "Resistor"
-			(at 341.63 67.31 0)
+			(at 340.36 57.15 0)
 			(effects
 				(font
@@
 	(symbol
 		(lib_id "Device:R")
-		(at 336.55 67.31 0)
+		(at 335.28 57.15 0)
 		(unit 1)
 		(exclude_from_sim no)
@@
 		(dnp no)
 		(property "Reference" "R20"
-			(at 330.454 66.294 0)
+			(at 329.184 56.134 0)
 			(effects
 				(font
@@
 		)
 		(property "Value" "5K"
-			(at 330.454 68.834 0)
+			(at 329.184 58.674 0)
 			(effects
 				(font
@@
 		)
 		(property "Footprint" "Resistor_SMD:R_0402_1005Metric"
-			(at 334.772 67.31 90)
+			(at 333.502 57.15 90)
 			(effects
 				(font
@@
 		)
 		(property "Datasheet" "~"
-			(at 336.55 67.31 0)
+			(at 335.28 57.15 0)
 			(effects
 				(font
@@
 		)
 		(property "Description" "Resistor"
-			(at 336.55 67.31 0)
+			(at 335.28 57.15 0)
 			(effects
 				(font
@@
 	(symbol
 		(lib_id "power:VCC")
-		(at 339.09 59.69 0)
+		(at 337.82 49.53 0)
 		(unit 1)
 		(exclude_from_sim no)
@@
 		(fields_autoplaced yes)
 		(property "Reference" "#PWR040"
-			(at 339.09 63.5 0)
+			(at 337.82 53.34 0)
 			(effects
 				(font
@@
 		)
 		(property "Value" "VCC"
-			(at 339.09 54.61 0)
+			(at 337.82 44.45 0)
 			(effects
 				(font
@@
 		)
 		(property "Footprint" ""
-			(at 339.09 59.69 0)
+			(at 337.82 49.53 0)
 			(effects
 				(font
@@
 		)
 		(property "Datasheet" ""
-			(at 339.09 59.69 0)
+			(at 337.82 49.53 0)
 			(effects
 				(font
@@
 		)
 		(property "Description" "Power symbol creates a global label with name \"VCC\""
-			(at 339.09 59.69 0)
+			(at 337.82 49.53 0)
 			(effects
 				(font
